File: Eagle/6WLS-30W.brd (EAGLE design)
At the start: 409.3 x 131.1 mm, 36 parts, among them J1 12VDC-8A, SW1 SPDTTHRU, U1 DCDCMULT6, U2 DCDCMULT6, U3 DCDCMULT6

Commit message: Larger copper pads for supply pins.
Switch to larger, oblong pads for supply pins. Thanks to Prism Circuits.
Parts:
- added X1: MKDSN1,5/2-5,08, con-phoenix-508:MKDSN1,5/2-5,08
Connections:
- net GND: now also X1.1, X1.2
Routing:
- net GND: track 50.2 -> 52.8 mm
- net 15V+: track 763.5 -> 764.6 mm
- net QGND: vias 9 -> 8
Other:
- board text removed: "BANANA"
Changed lines of the file:
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@@
 <wire x1="401.32" y1="0" x2="353.06" y2="0" width="0.0254" layer="20"/>
 <text x="326.6186" y="14.6939" size="1.27" layer="26" font="vector" ratio="12" rot="MR0">I2C PULLUPS </text>
-<text x="285.4198" y="71.3359" size="1.27" layer="26" font="vector" ratio="12" rot="MR0">GND</text>
-<text x="285.4198" y="69.6595" size="1.27" layer="26" font="vector" ratio="12" rot="MR0">BANANA</text>
+<text x="287.2232" y="64.008" size="1.27" layer="26" font="vector" ratio="12" rot="MR0">GND</text>
 <wire x1="401.32" y1="123.19" x2="401.32" y2="101.6" width="0.0254" layer="20"/>
 <wire x1="401.32" y1="101.6" x2="393.7" y2="93.98" width="0.0254" layer="20"/>
@@
 <vertex x="254.5334" y="71.6407"/>
 </polygon>
+<text x="292.735" y="64.008" size="1.27" layer="26" font="vector" ratio="12" rot="MR0">GND</text>
 </plain>
 <attributes>
@@
 <attribute name="VALUE" x="322.8848" y="115.316" size="1.27" layer="27" font="vector" ratio="12" rot="R90"/>
 </element>
+<element name="X1" library="con-phoenix-508" package="MKDSN1,5/2-5,08" value="MKDSN1,5/2-5,08" x="288.29" y="69.85" smashed="yes" rot="MR180"/>
 </elements>
 <signals>
@@
 <via x="349.25" y="69.914771875" extent="1-16" drill="1.2"/>
 <wire x1="349.25" y1="69.914771875" x2="349.25" y2="77.566521875" width="2.54" layer="16"/>
-<via x="288.29" y="71.184771875" extent="1-16" drill="2.95" diameter="5.08"/>
 <contactref element="C8" pad="-"/>
 <contactref element="C9" pad="+"/>
@@
 <contactref element="U2" pad="VO1-"/>
 <contactref element="U3" pad="VO1+"/>
-<wire x1="288.29" y1="71.184771875" x2="288.29" y2="71.12" width="5.08" layer="16"/>
 <contactref element="U2" pad="VO-"/>
 <wire x1="254" y1="30.48" x2="252.73" y2="1.2065" width="0" layer="19" extent="16-16"/>
 <wire x1="266.7" y1="30.48" x2="254" y2="30.48" width="0" layer="19" extent="1-1"/>
 <wire x1="252.73" y1="69.914771875" x2="254" y2="30.48" width="0" layer="19" extent="1-1"/>
-<wire x1="288.29" y1="71.184771875" x2="252.73" y2="69.914771875" width="0" layer="19" extent="1-1"/>
-<wire x1="349.25" y1="69.914771875" x2="288.29" y2="71.184771875" width="0" layer="19" extent="1-1"/>
-<wire x1="350.3676" y1="6.35" x2="349.25" y2="69.914771875" width="0" layer="19" extent="1-1"/>
-<wire x1="349.25" y1="1.2065" x2="350.3676" y2="6.35" width="0" layer="19" extent="16-16"/>
-<wire x1="336.2452" y1="6.35" x2="349.25" y2="1.2065" width="0" layer="19" extent="16-16"/>
 <wire x1="185.42" y1="50.8" x2="252.73" y2="69.914771875" width="0" layer="19" extent="1-1"/>
 <wire x1="172.72" y1="40.64" x2="185.42" y2="50.8" width="0" layer="19" extent="1-1"/>
 <wire x1="161.29" y1="1.2065" x2="172.72" y2="40.64" width="0" layer="19" extent="16-16"/>
+<wire x1="336.2452" y1="6.35" x2="266.7" y2="30.48" width="0" layer="19" extent="1-1"/>
+<wire x1="349.25" y1="1.2065" x2="336.2452" y2="6.35" width="0" layer="19" extent="16-16"/>
+<wire x1="350.3676" y1="6.35" x2="349.25" y2="1.2065" width="0" layer="19" extent="16-16"/>
+<wire x1="349.25" y1="69.914771875" x2="350.3676" y2="6.35" width="0" layer="19" extent="1-1"/>
 <wire x1="62.23" y1="-6.4135" x2="161.29" y2="-6.4135" width="0" layer="19" extent="16-16"/>
 <wire x1="62.23" y1="69.914771875" x2="62.23" y2="1.2065" width="0" layer="19" extent="1-16"/>
@@
 <wire x1="337.3628" y1="66.04" x2="337.3628" y2="69.914771875" width="1.778" layer="16"/>
 <wire x1="350.52" y1="66.04" x2="337.3628" y2="66.04" width="1.778" layer="15"/>
-<wire x1="337.3628" y1="66.04" x2="285.75" y2="66.04" width="1.778" layer="15"/>
-<wire x1="265.8618" y1="69.0118" x2="282.7782" y2="69.0118" width="1.778" layer="15"/>
-<wire x1="282.7782" y1="69.0118" x2="285.75" y2="66.04" width="1.778" layer="15"/>
+<wire x1="337.3628" y1="66.04" x2="283.21" y2="66.04" width="1.778" layer="15"/>
+<wire x1="265.8618" y1="69.0118" x2="280.2382" y2="69.0118" width="1.778" layer="15"/>
+<wire x1="280.2382" y1="69.0118" x2="283.21" y2="66.04" width="1.778" layer="15"/>
 <wire x1="265.8618" y1="69.0118" x2="262.89" y2="66.04" width="1.778" layer="15"/>
 <wire x1="262.89" y1="66.04" x2="246.38" y2="66.04" width="1.778" layer="15"/>
@@
 <wire x1="329.438" y1="69.85" x2="329.4634" y2="69.85" width="2.54" layer="2"/>
 <wire x1="349.2754" y1="69.8754" x2="349.3008" y2="69.8754" width="2.54" layer="2"/>
-<wire x1="289.56" y1="71.12" x2="287.02" y2="71.12" width="5.08" layer="2"/>
+<wire x1="290.83" y1="69.85" x2="285.75" y2="69.85" width="5.08" layer="2"/>
 <wire x1="389.001" y1="117.221" x2="390.779" y2="117.221" width="3.81" layer="2"/>
 <wire x1="350.3422" y1="6.2738" x2="350.3168" y2="6.2738" width="2.54" layer="2"/>
@@
 <wire x1="397.51" y1="112.22" x2="392.43" y2="117.3" width="2.54" layer="16"/>
 <wire x1="397.51" y1="106.68" x2="397.51" y2="112.22" width="2.54" layer="16"/>
+<contactref element="X1" pad="1"/>
+<contactref element="X1" pad="2"/>
 <wire x1="232.918" y1="1.1938" x2="252.7046" y2="1.1938" width="0" layer="19" extent="2-2"/>
 <wire x1="254" y1="30.48" x2="252.7046" y2="1.1938" width="0" layer="19" extent="2-2"/>
+<wire x1="290.83" y1="69.85" x2="290.8089" y2="69.825" width="0" layer="19" extent="1-2"/>
 <wire x1="329.438" y1="69.85" x2="325.12" y2="63.5" width="0" layer="19" extent="1-2"/>
 <wire x1="349.2754" y1="69.8754" x2="329.4634" y2="69.85" width="0" layer="19" extent="2-2"/>
@@
 <wire x1="349.2246" y1="1.1938" x2="336.2452" y2="6.3754" width="0" layer="19" extent="2-2"/>
 <wire x1="350.3422" y1="6.2738" x2="349.25" y2="1.1938" width="0" layer="19" extent="2-2"/>
-<wire x1="287.02" y1="71.12" x2="287.02" y2="38.1" width="0" layer="19" extent="1-2"/>
-<wire x1="252.7554" y1="69.9262" x2="287.02" y2="71.12" width="0" layer="19" extent="2-2"/>
+<wire x1="252.7554" y1="69.9262" x2="285.7289" y2="69.825" width="0" layer="19" extent="1-2"/>
 <wire x1="232.9434" y1="69.9262" x2="252.73" y2="69.9262" width="0" layer="19" extent="2-2"/>
 <wire x1="161.29" y1="1.27" x2="172.72" y2="40.64" width="0" layer="19" extent="2-2"/>
@@
 <wire x1="244.8052" y1="69.914771875" x2="244.8052" y2="77.566521875" width="2.54" layer="1"/>
 <wire x1="244.8052" y1="1.2065" x2="244.8052" y2="6.0452" width="1.778" layer="16"/>
-<wire x1="244.8052" y1="6.0452" x2="256.54" y2="17.78" width="1.778" layer="16"/>
+<wire x1="244.8052" y1="6.0452" x2="257.81" y2="19.05" width="1.778" layer="16"/>
 <wire x1="244.8052" y1="69.914771875" x2="244.8052" y2="61.2648" width="1.778" layer="16"/>
 <wire x1="341.3252" y1="1.2065" x2="341.3252" y2="-6.4135" width="2.54" layer="1"/>
@@
 <wire x1="242.57" y1="52.07" x2="254" y2="40.64" width="3.81" layer="15"/>
 <wire x1="254" y1="52.07" x2="254" y2="40.64" width="1.778" layer="16"/>
-<wire x1="256.54" y1="17.78" x2="256.54" y2="38.1" width="1.778" layer="16"/>
-<wire x1="256.54" y1="38.1" x2="254" y2="40.64" width="1.778" layer="16"/>
+<wire x1="257.81" y1="19.05" x2="257.81" y2="36.83" width="1.778" layer="16"/>
+<wire x1="257.81" y1="36.83" x2="254" y2="40.64" width="1.778" layer="16"/>
 </signal>
 <signal name="NGND">
@@
 </signal>
 <signal name="COM">
+<contactref element="U1" pad="TRIM1"/>
 <contactref element="U1" pad="TRIM"/>
-<contactref element="U1" pad="TRIM1"/>
+<contactref element="U2" pad="TRIM1"/>
 <contactref element="U2" pad="TRIM"/>
-<contactref element="U2" pad="TRIM1"/>
+<contactref element="U3" pad="TRIM1"/>
 <contactref element="U3" pad="TRIM"/>
-<contactref element="U3" pad="TRIM1"/>
 <wire x1="172.72" y1="20.32" x2="185.42" y2="40.64" width="0" layer="19" extent="1-1"/>
 <wire x1="254" y1="20.32" x2="185.42" y2="40.64" width="0" layer="19" extent="1-1"/>
