File: Eagle/6WLS-40W-OTHER.brd (EAGLE design)
At the start: 381.3 x 87 mm, 26 parts, among them U1 DCDCEC7C01, U2 DCDCEC7C03, U3 DCDCEC7C03, X1 MKDSN1,5/5-5,08

Commit message: Larger copper pads for supply pins.
Switch to larger, oblong pads for supply pins. Thanks to Prism Circuits.
Other:
- board text added: "6WLS-40W-OTHER R1 11/24 DC (WITH THANKS TO D. BROWN)"
- board text removed: "6WLS-40W-OTHER R0 3/23 DC (WITH THANKS TO D. BROWN)"
Changed lines of the file:
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@@
 <plain>
 <text x="118.364" y="32.3469" size="6.096" layer="26" font="vector" ratio="12" rot="MR0">STUDIOHSOFTWARE.COM</text>
-<text x="109.474" y="29.1465" size="1.778" layer="26" font="vector" ratio="12" rot="MR0">6WLS-40W-OTHER R0 3/23 DC  (WITH THANKS TO D. BROWN)</text>
+<text x="109.474" y="29.1465" size="1.778" layer="26" font="vector" ratio="12" rot="MR0">6WLS-40W-OTHER R1 11/24 DC  (WITH THANKS TO D. BROWN)</text>
 <wire x1="48.26" y1="0" x2="48.26" y2="-7.9375" width="0.0254" layer="20"/>
 <wire x1="48.26" y1="-7.9375" x2="22.606" y2="-7.9375" width="0.0254" layer="20"/>
