File: Eagle/6WLS-40W-OTHER.sch (EAGLE design)
At the start: 26 parts, among them U1 DCDCEC7C01, U2 DCDCEC7C03, U3 DCDCEC7C03, X1 MKDSN1,5/5-5,08

Commit message: Larger copper pads for supply pins.
Switch to larger, oblong pads for supply pins. Thanks to Prism Circuits.
Other:
- note added: "1"
- note added: "FBA-6WLS-40W-OTHER"
- note removed: "9"
- note removed: "FBA-6WLS-40W"
Changed lines of the file:
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@@
 <sheet>
 <plain>
-<text x="367.03" y="6.35" size="2.54" layer="97" font="vector" ratio="12">FBA-6WLS-40W</text>
-<text x="417.83" y="6.35" size="2.54" layer="97" font="vector" ratio="12">9</text>
+<text x="367.03" y="6.35" size="2.54" layer="97" font="vector" ratio="12">FBA-6WLS-40W-OTHER</text>
+<text x="417.83" y="6.35" size="2.54" layer="97" font="vector" ratio="12">1</text>
 </plain>
 <instances>
