File: Eagle/6WLS-40W.sch (EAGLE design)
At the start: 36 parts, among them J1 12VDC-8A, SW1 SPDTTHRU, U1 DCDCEC7C01, U2 DCDCEC7C03, U3 DCDCEC7C03

Commit message: Larger copper pads for supply pins.
Switch to larger, oblong pads for supply pins. Thanks to Prism Circuits.
Parts:
- added X1: MKDSN1,5/2-5,08, con-phoenix-508:MKDSN1,5/2-5,08
Connections:
- net GND: now also X1-1.KL, X1-2.KL
Other:
- note added: "3"
- note removed: "9"
Changed lines of the file:
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@@
 <part name="SW1" library="studio_h" deviceset="SPDT" device="THRU"/>
 <part name="SV1" library="studio_h" deviceset="MA06-2" device="CARD"/>
+<part name="X1" library="con-phoenix-508" deviceset="MKDSN1,5/2-5,08" device=""/>
 </parts>
 <sheets>
@@
 <plain>
 <text x="367.03" y="6.35" size="2.54" layer="97" font="vector" ratio="12">FBA-6WLS-40W</text>
-<text x="417.83" y="6.35" size="2.54" layer="97" font="vector" ratio="12">9</text>
+<text x="417.83" y="6.35" size="2.54" layer="97" font="vector" ratio="12">3</text>
 </plain>
 <instances>
@@
 <instance part="SW1" gate="G$1" x="218.44" y="248.92"/>
 <instance part="SV1" gate="1" x="172.72" y="220.98"/>
+<instance part="X1" gate="-1" x="58.42" y="195.58"/>
+<instance part="X1" gate="-2" x="58.42" y="190.5"/>
 </instances>
 <busses>
@@
 <junction x="53.34" y="55.88"/>
 </segment>
-</net>
+<segment>
+<label x="55.88" y="180.34" size="1.27" layer="95" font="vector" ratio="12" xref="yes"/>
+<pinref part="X1" gate="-1" pin="KL"/>
+<wire x1="55.88" y1="195.58" x2="50.8" y2="195.58" width="0.1524" layer="91"/>
+<wire x1="50.8" y1="195.58" x2="50.8" y2="190.5" width="0.1524" layer="91"/>
+<wire x1="50.8" y1="190.5" x2="50.8" y2="180.34" width="0.1524" layer="91"/>
+<wire x1="50.8" y1="180.34" x2="55.88" y2="180.34" width="0.1524" layer="91"/>
+<pinref part="X1" gate="-2" pin="KL"/>
+<wire x1="55.88" y1="190.5" x2="50.8" y2="190.5" width="0.1524" layer="91"/>
+<junction x="50.8" y="190.5"/>
+</segment>
+</net>
